File: TeaTemperaturePCB.kicad_pcb (KiCad board)
At the start: 2 copper layers, 24 x 43 mm, 12 parts, among them Q1 SI2323DDS-T1-GE3, Q2 BC847B, Q3 SSM3K35AMFV, SW1 LL3301FF065QJ, SW2 LL3301FF065QJ, U1 BAT-HLD-001, U2 STM32L011K4T6, U3 ABT-407-RC, U4 LMT84LPGM, U5 TDSR0760, U6 TDSR0760, U7 AP7354D-18W5-7

Commit message: Added kicad project
Parts:
- added C1: 0.1uF, Capacitors_SMD:C_0603, F.Cu at (160.8, 100.2)
- added C2: 0.1uF, Capacitors_SMD:C_0603, F.Cu at (155.8, 104.3)
- added C3: 0.1uF, Capacitors_SMD:C_0603, F.Cu at (160.8, 101.8)
- added C4: 0.1uF, Capacitors_SMD:C_0603, F.Cu at (165.3, 99.8)
- added C5: 10uF, Capacitors_SMD:C_0603, F.Cu at (165.3, 101.4)
- added D1: S1G-K R2G, Diodes_SMD:SMA_Handsoldering, F.Cu at (154.4, 99.8)
- added Q4: SSM3K35AMFV, custom_footprints:SOT-723, F.Cu at (170.1, 101.5)
- added R1: 250K, Resistors_SMD:R_0603, F.Cu at (151.9, 102.7)
- added R10: 750, Resistors_SMD:R_0603, F.Cu at (164.5, 137.7)
- added R11: 750, Resistors_SMD:R_0603, F.Cu at (190.5, 139.7)
- added R12: 750, Resistors_SMD:R_0603, F.Cu at (166.2, 137.7)
- added R13: 750, Resistors_SMD:R_0603, F.Cu at (162.9, 133.6)
- added R14: 750, Resistors_SMD:R_0603, F.Cu at (167.6, 152.4)
- added R15: 750, Resistors_SMD:R_0603, F.Cu at (164.5, 133.6)
- added R16: 750, Resistors_SMD:R_0603, F.Cu at (165.9, 148.4)
- added R17: 750, Resistors_SMD:R_0603, F.Cu at (166.2, 133.6)
- added R18: 750, Resistors_SMD:R_0603, F.Cu at (169.2, 152.4)
- added R19: 750, Resistors_SMD:R_0603, F.Cu at (167.6, 148.4)
- added R2: 10K, Resistors_SMD:R_0603, F.Cu at (160.9, 98.6)
- added R20: 750, Resistors_SMD:R_0603, F.Cu at (170.9, 152.4)
- added R21: 10K, Resistors_SMD:R_0603, F.Cu at (168.1, 99.9)
- added R22: 250K, Resistors_SMD:R_0603, F.Cu at (165.2, 103.0)
- added R23: 10K, Resistors_SMD:R_0603, F.Cu at (168.1, 101.5)
- added R24: 250K, Resistors_SMD:R_0603, F.Cu at (170.8, 99.9)
- added R25: 250K, Resistors_SMD:R_0603, F.Cu at (167.8, 103.2)
- added R3: 250K, Resistors_SMD:R_0603, F.Cu at (155.9, 102.7)
- added R4: 10K, Resistors_SMD:R_0603, F.Cu at (151.9, 104.3)
- added R5: 750, Resistors_SMD:R_0603, F.Cu at (166.4, 107.2)
- added R6: 750, Resistors_SMD:R_0603, F.Cu at (161.2, 137.7)
- added R7: 750, Resistors_SMD:R_0603, F.Cu at (187.5, 148.9)
- added R8: 750, Resistors_SMD:R_0603, F.Cu at (162.9, 137.7)
- added R9: 750, Resistors_SMD:R_0603, F.Cu at (161.2, 133.6)
- Q2: value BC847B -> SSM3K35AMFV; footprint TO_SOT_Packages_SMD:SOT-23 -> custom_footprints:SOT-723
- moved U2 31.8 mm to (183.7, 149.8)
- moved U1 23.8 mm to (162.6, 157.4)
- moved SW1 23.7 mm to (156.1, 145.4)
- moved U3 23.7 mm to (153.6, 140.4)
- moved U5 23.7 mm to (169.1, 144.4)
- moved Q2 6.48 mm to (154.9, 108.0)
- moved Q1 3.59 mm to (161.3, 105.4)
- moved Q3 2.41 mm to (152.4, 107.5)
Connections:
- net Net-(SW1-Pad2) renamed /BTN_UP
- net Net-(SW2-Pad2) renamed /BTN_DN
- net Net-(U2-Pad23) renamed /SWDIO
- net Net-(U2-Pad24) renamed /SWCLK
- net Net-(U2-Pad25) renamed /VCP_RX
- net Net-(U2-Pad4) renamed /NRST
- net Net-(U2-Pad8) renamed /VCP_TX
- net Net-(U4-Pad2) renamed /THERM_MEAS
- Q1 pad 1: Net-(Q1-Pad1) -> GND
- Q1 pad 2: Net-(Q1-Pad2) -> +BATT
- Q1 pad 3: Net-(Q1-Pad3) -> VCC
- Q2 pad 2: Net-(Q2-Pad2) -> GND
- Q2 pad 3: Net-(Q2-Pad3) -> Net-(D1-Pad2)
- Q3 pad 2: Net-(Q3-Pad2) -> GND
- SW1 pad 1: Net-(SW1-Pad1) -> VCC
- SW2 pad 1: Net-(SW2-Pad1) -> VCC
- U2 pad 1: Net-(U2-Pad1) -> VCC
- U2 pad 14: Net-(U2-Pad14) -> /DISP_SEG_B
- U2 pad 15: Net-(U2-Pad15) -> /DISP_SEG_E
- U2 pad 16: Net-(U2-Pad16) -> GND
- U2 pad 17: Net-(U2-Pad1) -> VCC
- U2 pad 18: Net-(U2-Pad18) -> /DISP_SEG_F
- U2 pad 2: Net-(U2-Pad2) -> /MCO
- U2 pad 21: Net-(U2-Pad21) -> /DISP_SEG_G
- U2 pad 22: Net-(U2-Pad22) -> /DISP_SEG_A
- U2 pad 28: Net-(U2-Pad28) -> /DISP_SEG_DP
- U2 pad 29: Net-(U2-Pad29) -> /DISP_SEG_D
- U2 pad 30: Net-(U2-Pad30) -> /DISP_SEG_C
- U2 pad 32: Net-(U2-Pad16) -> GND
- U2 pad 5: Net-(U2-Pad5) -> +1V8
- U2 pad 6: Net-(U2-Pad6) -> /MCO
- U3 pad 1: Net-(U3-Pad1) -> VCC
- U3 pad 2: Net-(U3-Pad2) -> Net-(D1-Pad2)
- U4 pad 1: Net-(U4-Pad1) -> Net-(Q3-Pad3)
- U4 pad 3: Net-(U4-Pad3) -> +1V8
- U5 pad 3: Net-(U5-Pad3) -> /DISP_BLK_1_EN
- U5 pad 8: Net-(U5-Pad8) -> /DISP_BLK_1_EN
- U6 pad 3: Net-(U6-Pad3) -> /DISP_BLK_2_EN
- U6 pad 8: Net-(U6-Pad8) -> /DISP_BLK_2_EN
- U7 pad 1: Net-(U7-Pad1) -> VCC
- U7 pad 2: Net-(U7-Pad2) -> GND
- U7 pad 3: Net-(U7-Pad3) -> VCC
- U7 pad 5: Net-(U7-Pad5) -> +1V8
Other:
- board size 24 x 43 mm -> 30.3 x 65.9 mm
