File: TeaTemperaturePCB.sch (KiCad schematic (older format))
At the start: 12 parts, among them Q1 SI2323DDS-T1-GE3, Q2 BC847B, Q3 SSM3K35AMFV, SW1 LL3301FF065QJ, SW2 LL3301FF065QJ, U1 BAT-HLD-001, U2 STM32L011K4T6, U3 ABT-407-RC, U4 LMT84LPGM, U5 TDSR0760, U6 TDSR0760, U7 AP7354D-18W5-7

Commit message: Added kicad project
Parts:
- removed Q2: BC847B, TO_SOT_Packages_SMD:SOT-23, symbol Device:Q_NPN_BEC
- added C1, C2, C3, C4: 0.1uF, Capacitors_SMD:C_0603, symbol Device:C
- added C5, C? (x2): 10uF, Capacitors_SMD:C_0603, symbol Device:C
- added D1: S1G-K R2G, Diodes_SMD:SMA_Handsoldering, symbol Device:D_ALT
- added J?: Con_programmer, symbol Connector_Generic:Conn_02x03_Counter_Clockwise
- added Q2, Q4: SSM3K35AMFV, custom_footprints:SOT-723, symbol Device:Q_NMOS_GSD
- added R1, R22, R24, R25, R3, R?: 250K, Resistors_SMD:R_0603, symbol Device:R
- added R10, R11, R12, R13, R14, R15, R16, R17, R18, R19, R20, R5, R6, R7, R8, R9: 750, Resistors_SMD:R_0603, symbol Device:R
- added R2, R21, R23, R4: 10K, Resistors_SMD:R_0603, symbol Device:R
- added R? (x2): 250000K, Resistors_SMD:R_0603, symbol Device:R
Connections:
- net +BATT: now also Q1.2 (S)
- net GND: now also Q1.1 (G), Q3.2 (S), U2.16 (VSS), U2.32 (VSS), U7.2 (GND), C1.2, C2.2, C3.2, C4.2, C5.2, C?.2, C?.2, Q2.2 (S), Q4.2 (S), R1.1, R21.1, R22.1, R3.1, R?.2
- net VCC: now reaches U2.1 (VDD), U2.17 (VDD)
- net VCC: now also Q1.3 (D), SW1.1, SW2.1, U3.1 (+), U7.1 (IN), U7.3 (EN), C1.1, C4.1, C5.1, D1.1 (K), R24.2, R?.1
- net DISP_BLK_2_EN: now reaches U2.10 (PA4)
- net DISP_BLK_2_EN: now also U6.3 (CC), U6.8 (CC)
- net THERM_CTRL: now reaches U2.11 (PA5)
- net THERM_CTRL: now also R3.2, R4.2
- net BATT_MEAS: now reaches U2.12 (PA6)
- net BATT_MEAS: now also R24.1, R25.2
- net BATT_MEAS_CTRL: now reaches U2.13 (PA7)
- net BATT_MEAS_CTRL: now also R22.2, R23.2
- net DISP_SEG_B: now reaches U2.14 (PB0)
- net DISP_SEG_B: now also R14.2, R6.2
- net DISP_SEG_E: now reaches U2.15 (PB1)
- net DISP_SEG_E: now also R17.2, R9.2
- net DISP_SEG_F: now reaches U2.18 (PA8)
- net DISP_SEG_F: now also R10.2, R18.2
- net MCO: now reaches U2.2 (PC14-OSC32_IN)
- net DISP_SEG_G: now reaches U2.21 (PA11)
- net DISP_SEG_G: now also R11.2, R19.2
- net DISP_SEG_A: now reaches U2.22 (PA12)
- net DISP_SEG_A: now also R13.2, R5.2
- net SWDIO: now reaches U2.23 (PA13)
- net SWCLK: now reaches U2.24 (PA14)
- net VCP_RX: now reaches U2.25 (PA15)
- net DISP_BLK_1_EN: now reaches U2.27 (PB4)
- net DISP_BLK_1_EN: now also U5.3 (CC), U5.8 (CC)
- net DISP_SEG_DP: now reaches U2.28 (PB5)
- net DISP_SEG_DP: now also R12.2, R20.2
- net DISP_SEG_D: now reaches U2.29 (PB6)
- net DISP_SEG_D: now also R16.2, R8.2
- net DISP_SEG_C: now reaches U2.30 (PB7)
- net DISP_SEG_C: now also R15.2, R7.2
- net at U2.31 (PB9-BOOT0): now also R21.2
- net NRST: now reaches U2.4 (NRST)
- net +1V8: now reaches U2.5 (VDDA)
- net +1V8: now also U4.3 (Vdd), U7.5 (OUT), C2.1, C3.1
- net BTN_UP: now reaches U2.6 (PA0-CK_IN)
- net BTN_UP: now also SW1.2
- net THERM_MEAS: now reaches U2.7 (PA1)
- net THERM_MEAS: now also U4.2 (OUT)
- net BTN_DN: now reaches U2.8 (PA2)
- net BTN_DN: now also SW2.2
- net BUZZER_CTRL: now reaches U2.9 (PA3)
- net BUZZER_CTRL: now also R1.2, R2.2
- net at U3.2 (-): now also D1.2 (A), Q2.3 (D)
- net at U4.1 (GND): now also Q3.3 (D)
- net at U5.1 (E): now also R17.1
- net at U5.10 (F): now also R18.1
- net at U5.2 (D): now also R16.1
- net at U5.4 (C): now also R15.1
- net at U5.5 (DP): now also R20.1
- net at U5.6 (B): now also R14.1
- net at U5.7 (A): now also R13.1
- net at U5.9 (G): now also R19.1
- net at U6.1 (E): now also R9.1
- net at U6.10 (F): now also R10.1
- net at U6.2 (D): now also R8.1
- net at U6.4 (C): now also R7.1
- net at U6.5 (DP): now also R12.1
- net at U6.6 (B): now also R6.1
- net at U6.7 (A): now also R5.1
- net at U6.9 (G): now also R11.1
- net at Q3.1 (G): now also R4.1
- new net: Q2.1 (G), R2.1
- new net: R?.1, R?.2
- new net: C?.1, R?.2
- new net: C?.1, R?.1
- new net: Q4.1 (G), R23.1
- new net: Q4.3 (D), R25.1
Other:
- moved on the sheet: Q1, Q3, SW1, SW2, U2, U3, U5, U6, U7
