File: _autosave-TeaTemperaturePCB.kicad_pcb (KiCad board)
At the start: 2 copper layers, 24 x 43 mm, 44 parts, among them Q1 SI2323DDS-T1-GE3, Q2 SSM3K35AMFV, Q3 SSM3K35AMFV, Q4 SSM3K35AMFV, SW1 LL3301FF065QJ, SW2 LL3301FF065QJ, U1 BAT-HLD-001, U2 STM32L011K4T6, U3 ABT-407-RC, U4 LMT84LPGM, U5 TDSR0760, U6 TDSR0760, U7 AP7354D-18W5-7

Commit message: Added kicad project
Parts:
- moved R12 23.7 mm to (159.8, 114.8)
- moved R7 23.7 mm to (181.2, 126.0)
- moved R10 23.7 mm to (158.2, 114.8)
- moved R6 23.7 mm to (154.9, 114.8)
- moved R8 23.7 mm to (156.5, 114.8)
- moved U2 23.7 mm to (177.4, 127.0)
- moved R17 23.7 mm to (159.8, 110.8)
- moved R13 23.7 mm to (156.5, 110.8)
- moved R15 23.7 mm to (158.2, 110.8)
- moved R9 23.7 mm to (154.9, 110.8)
- moved R11 23.7 mm to (184.2, 116.8)
Changed lines of the file:
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@@
   )
   (module STM32L011K4T6:QFP80P900X900X160-32N (layer F.Cu)
-    (at 183.72 149.83)
+    (at 177.37 126.97)
     (attr smd)
     (fp_text reference U2 (at -2.51569 -6.35035) (layer F.SilkS)
@@
   )
   (module Resistors_SMD:R_0603 (layer F.Cu)
-    (at 161.225001 137.674999 90)
+    (at 154.875001 114.814999 90)
     (descr "Resistor SMD 0603, reflow soldering, Vishay (see dcrcw.pdf)")
     (tags "resistor 0603")
@@
   )
   (module Resistors_SMD:R_0603 (layer F.Cu)
-    (at 187.515001 148.864999 90)
+    (at 181.165001 126.004999 90)
     (descr "Resistor SMD 0603, reflow soldering, Vishay (see dcrcw.pdf)")
     (tags "resistor 0603")
@@
   )
   (module Resistors_SMD:R_0603 (layer F.Cu)
-    (at 162.875001 137.674999 90)
+    (at 156.525001 114.814999 90)
     (descr "Resistor SMD 0603, reflow soldering, Vishay (see dcrcw.pdf)")
     (tags "resistor 0603")
@@
   )
   (module Resistors_SMD:R_0603 (layer F.Cu)
-    (at 161.225001 133.624999 90)
+    (at 154.875001 110.764999 90)
     (descr "Resistor SMD 0603, reflow soldering, Vishay (see dcrcw.pdf)")
     (tags "resistor 0603")
@@
   )
   (module Resistors_SMD:R_0603 (layer F.Cu)
-    (at 164.525001 137.674999 90)
+    (at 158.175001 114.814999 90)
     (descr "Resistor SMD 0603, reflow soldering, Vishay (see dcrcw.pdf)")
     (tags "resistor 0603")
@@
   )
   (module Resistors_SMD:R_0603 (layer F.Cu)
-    (at 190.5 139.7 90)
+    (at 184.15 116.84 90)
     (descr "Resistor SMD 0603, reflow soldering, Vishay (see dcrcw.pdf)")
     (tags "resistor 0603")
@@
   )
   (module Resistors_SMD:R_0603 (layer F.Cu)
-    (at 166.175001 137.674999 90)
+    (at 159.825001 114.814999 90)
     (descr "Resistor SMD 0603, reflow soldering, Vishay (see dcrcw.pdf)")
     (tags "resistor 0603")
@@
   )
   (module Resistors_SMD:R_0603 (layer F.Cu)
-    (at 162.875001 133.624999 90)
+    (at 156.525001 110.764999 90)
     (descr "Resistor SMD 0603, reflow soldering, Vishay (see dcrcw.pdf)")
     (tags "resistor 0603")
@@
   )
   (module Resistors_SMD:R_0603 (layer F.Cu)
-    (at 164.525001 133.624999 90)
+    (at 158.175001 110.764999 90)
     (descr "Resistor SMD 0603, reflow soldering, Vishay (see dcrcw.pdf)")
     (tags "resistor 0603")
@@
   )
   (module Resistors_SMD:R_0603 (layer F.Cu)
-    (at 166.175001 133.624999 90)
-    (descr "Resistor SMD 0603, reflow soldering, Vishay (see dcrcw.pdf)")
-    (tags "resistor 0603")
+    (at 159.825001 110.764999 90)
+    (descr "Resistor SMD 0603, reflow soldering, Vishay (see dcrcw.pdf)")
+    (tags "resistor 0603")
